Commit message: Add Go2 LiDAR sensor to Gazebo model

File: go2_description/xacro/gazebo.xacro (robot description, xacro)
@@ -125,4 +125,31 @@
             </sensor>
         </gazebo>
+		<gazebo reference="velodyne_frame">
+			<sensor name="velodyne" type="gpu_lidar">
+				<pose>0 0 0 0 0 0</pose>
+				<visualize>false</visualize>
+				<update_rate>10</update_rate>
+				<lidar>
+					<scan>
+						<horizontal>
+							<samples>440</samples>
+							<min_angle>-3.14159</min_angle>
+							<max_angle>3.14159</max_angle>
+						</horizontal>
+						<vertical>
+							<samples>16</samples>
+							<min_angle>-0.2618</min_angle>
+							<max_angle>0.2618</max_angle>
+						</vertical>
+					</scan>
+					<range>
+						<min>0.3</min>
+						<max>100.0</max>
+					</range>
+				</lidar>
+				<topic>/${robot_name}/velodyne_points</topic>
+				<gz_frame_id>velodyne_frame</gz_frame_id>
+			</sensor>
+		</gazebo>
         <gazebo reference="camera_face">
             <!-- <material>Gazebo/Black</material> -->

File: go2_description/xacro/robot.xacro (robot description, xacro)
@@ -82,4 +82,28 @@
         </collision>
     </link>
+	<joint name="velodyne_joint" type="fixed">
+		<parent link="base_link"/>
+		<child link="velodyne_frame"/>
+		<origin xyz="0.15 0.0 0.15" rpy="0 0 0" />
+	</joint>
+	<link name="velodyne_frame">
+		<inertial>
+			<mass value="0.083"/>
+			<origin rpy="0 0 0" xyz="0 0 0"/>
+			<inertia ixx="0.0001" ixy="0" ixz="0" iyy="0.0001" iyz="0" izz="0.0001"/>
+		</inertial>
+		<visual>
+			<origin rpy="0 0 0" xyz="0 0 0"/>
+			<geometry>
+				<cylinder length="0.07" radius="0.05" />
+			</geometry>
+		</visual>
+		<collision>
+			<origin rpy="0 0 0" xyz="0 0 0"/>
+			<geometry>
+				<cylinder length="0.07" radius="0.05" />
+			</geometry>
+		</collision>
+	</link>
     <joint name="imu_joint" type="fixed">
         <parent link="base_link"/>
